File: Control_MCU.kicad_sch (KiCad schematic)
At the start: 87 parts, among them Q31 BSS123, Q32 BSS123, Q33 BSS123, SW10 TS1701-CZ55HBS, SW11 TS1701-CZ55HBS, SW12 TS1701-CZ55HBS, SW13 TS1701-CZ55HBS, SW6 TS1701-CZ55HBS, SW7 TS1701-CZ55HBS, SW9 TS1701-CZ55HBS, U1 STM32G474VETx, U15 UAD8C05L01_C3001951, U16 UAD8C05L01_C3001951, U17 161N-4BVS11, U2 DSC1003DL2-008.0000T, U20 UAD8C05L01_C3001951, U21 UAD8C05L01_C3001951, U3 UAD8C05L01_C3001951

Commit message: Update rev1 PCB and schematics with existing project libraries
Parts:
- R148: value 0 -> 100M
Changed lines of the file:
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@@
 	)
 	(junction
-		(at 49.53 213.36)
+		(at 49.53 210.82)
 		(diameter 0)
 		(color 0 0 0 0)
@@
 	(wire
 		(pts
+			(xy 50.8 210.82) (xy 50.8 213.36)
+		)
+		(stroke
+			(width 0)
+			(type default)
+		)
+	)
+	(wire
+		(pts
 			(xy 43.18 114.3) (xy 45.72 114.3)
 		)
@@
 	(wire
 		(pts
-			(xy 49.53 209.55) (xy 49.53 213.36)
-		)
-		(stroke
-			(width 0)
-			(type default)
-		)
-	)
-	(wire
-		(pts
 			(xy 59.69 171.45) (xy 52.07 171.45)
 		)
@@
 	(wire
 		(pts
-			(xy 50.8 213.36) (xy 49.53 213.36)
+			(xy 50.8 210.82) (xy 49.53 210.82)
 		)
 		(stroke
@@
 	(wire
 		(pts
+			(xy 49.53 209.55) (xy 49.53 213.36)
+		)
+		(stroke
+			(width 0)
+			(type default)
+		)
+	)
+	(wire
+		(pts
 			(xy 250.19 38.1) (xy 240.03 38.1)
 		)
@@
 	(global_label "PB8_BOOT"
 		(shape passive)
-		(at 50.8 213.36 0)
+		(at 50.8 210.82 0)
 		(effects
 			(font
@@
 		)
 		(property "Intersheetrefs" "${INTERSHEET_REFS}"
-			(at 50.8 213.36 0)
+			(at 50.8 210.82 0)
 			(hide yes)
 			(show_name no)
@@
 			)
 		)
-		(property "Value" "0"
+		(property "Value" "100M"
 			(at 81.28 186.6899 0)
 			(show_name no)
