File: receiver.kicad_sch (KiCad schematic)
At the start: 96 parts, among them U10 SN74CBT3253, U11 SN74CBT3253, U12 TLV9062xD, U13 PCM1821QRTERQ1, U14 NE5532, U22 UAD8C05L01_C3001951, U23 UAD8C05L01_C3001951, U24 UAD8C05L01_C3001951, U9 TLV9062xD

Commit message: Update rev1 PCB and schematics with existing project libraries
Changed lines of the file:
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@@
 		(dnp no)
 		(property "Reference" "U14"
-			(at 148.59 132.0799 0)
+			(at 151.384 132.334 0)
 			(show_name no)
 			(do_not_autoplace no)
@@
 		)
 		(property "Value" "NE5532"
-			(at 148.59 134.6199 0)
+			(at 151.384 134.874 0)
 			(show_name no)
 			(do_not_autoplace no)
