File: untitled.kicad_sch (KiCad schematic)
At the start: 50 parts, among them Q1 APM4953_C5185739, Q13 BSS123, Q16 APM4953_C5185739, Q17 BSS123, Q2 APM4953_C5185739, SW8 TS1701-CZ55HBS, U18 161N-4BVS11, U19 LM1084IT-5.0G, U4 UZ1085L-33-TN3-R

Commit message: Update rev1 PCB and schematics with existing project libraries
Parts:
- added JP21: (no value), HansPinhead:1X02, symbol HansPinhead:PINHD-1X2
Connections:
- net VIN: now also JP21.2; no longer Q2.5 (D1), Q2.6 (D1)
- new net: JP21.1, Q2.5 (D1), Q2.6 (D1)
Other:
- moved on the sheet: R108
Changed lines of the file:
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@@
 	)
 	(junction
-		(at 115.57 121.92)
-		(diameter 0)
-		(color 0 0 0 0)
-	)
-	(junction
 		(at 187.96 95.25)
 		(diameter 0)
@@
 	)
 	(junction
+		(at 115.57 132.08)
+		(diameter 0)
+		(color 0 0 0 0)
+	)
+	(junction
 		(at 138.43 143.51)
 		(diameter 0)
@@
 	)
 	(junction
-		(at 115.57 132.08)
+		(at 114.3 120.65)
 		(diameter 0)
 		(color 0 0 0 0)
@@
 	(wire
 		(pts
-			(xy 41.91 106.68) (xy 45.72 106.68)
-		)
-		(stroke
-			(width 0)
-			(type default)
-		)
-	)
-	(wire
-		(pts
 			(xy 104.14 50.8) (xy 104.14 54.61)
 		)
@@
 	(wire
 		(pts
-			(xy 115.57 132.08) (xy 115.57 121.92)
-		)
-		(stroke
-			(width 0)
-			(type default)
-		)
-	)
-	(wire
-		(pts
 			(xy 95.25 128.27) (xy 95.25 132.08)
 		)
@@
 	(wire
 		(pts
+			(xy 121.92 120.65) (xy 114.3 120.65)
+		)
+		(stroke
+			(width 0)
+			(type default)
+		)
+	)
+	(wire
+		(pts
 			(xy 16.51 53.34) (xy 39.37 53.34)
 		)
@@
 	(wire
 		(pts
+			(xy 87.63 120.65) (xy 87.63 121.92)
+		)
+		(stroke
+			(width 0)
+			(type default)
+		)
+	)
+	(wire
+		(pts
 			(xy 99.06 85.09) (xy 99.06 92.71)
 		)
@@
 	(wire
 		(pts
-			(xy 115.57 121.92) (xy 115.57 106.68)
+			(xy 114.3 120.65) (xy 114.3 106.68)
 		)
 		(stroke
@@
 	(wire
 		(pts
+			(xy 115.57 132.08) (xy 121.92 132.08)
+		)
+		(stroke
+			(width 0)
+			(type default)
+		)
+	)
+	(wire
+		(pts
 			(xy 86.36 49.53) (xy 86.36 50.8)
 		)
@@
 	(wire
 		(pts
+			(xy 124.46 137.16) (xy 125.73 137.16)
+		)
+		(stroke
+			(width 0)
+			(type default)
+		)
+	)
+	(wire
+		(pts
 			(xy 24.13 101.6) (xy 24.13 109.22)
 		)
@@
 	(wire
 		(pts
-			(xy 115.57 132.08) (xy 115.57 134.62)
-		)
-		(stroke
-			(width 0)
-			(type default)
-		)
-	)
-	(wire
-		(pts
 			(xy 60.96 92.71) (xy 90.17 92.71)
 		)
@@
 	(wire
 		(pts
+			(xy 121.92 120.65) (xy 121.92 132.08)
+		)
+		(stroke
+			(width 0)
+			(type default)
+		)
+	)
+	(wire
+		(pts
 			(xy 163.83 64.77) (xy 163.83 54.61)
 		)
@@
 	(wire
 		(pts
+			(xy 43.18 106.68) (xy 41.91 106.68)
+		)
+		(stroke
+			(width 0)
+			(type default)
+		)
+	)
+	(wire
+		(pts
 			(xy 95.25 134.62) (xy 100.33 134.62)
 		)
@@
 	(wire
 		(pts
-			(xy 50.8 106.68) (xy 55.88 106.68)
+			(xy 48.26 106.68) (xy 55.88 106.68)
 		)
 		(stroke
@@
 	(wire
 		(pts
-			(xy 115.57 106.68) (xy 125.73 106.68)
+			(xy 114.3 106.68) (xy 125.73 106.68)
 		)
 		(stroke
@@
 	(wire
 		(pts
-			(xy 115.57 137.16) (xy 125.73 137.16)
+			(xy 115.57 137.16) (xy 119.38 137.16)
 		)
 		(stroke
@@
 	(wire
 		(pts
+			(xy 115.57 132.08) (xy 115.57 134.62)
+		)
+		(stroke
+			(width 0)
+			(type default)
+		)
+	)
+	(wire
+		(pts
 			(xy 11.43 43.18) (xy 11.43 50.8)
 		)
@@
 	(wire
 		(pts
-			(xy 87.63 121.92) (xy 115.57 121.92)
+			(xy 87.63 120.65) (xy 114.3 120.65)
 		)
 		(stroke
@@
 	(symbol
 		(lib_id "Device:R_Small")
-		(at 48.26 106.68 90)
+		(at 45.72 106.68 90)
 		(unit 1)
 		(body_style 1)
@@
 		(fields_autoplaced yes)
 		(property "Reference" "R108"
-			(at 48.26 101.6 90)
+			(at 45.72 101.6 90)
 			(show_name no)
 			(do_not_autoplace no)
@@
 		)
 		(property "Value" "0"
-			(at 48.26 104.14 90)
+			(at 45.72 104.14 90)
 			(show_name no)
 			(do_not_autoplace no)
@@
 		)
 		(property "Footprint" "Resistor_SMD:R_1206_3216Metric_Pad1.30x1.75mm_HandSolder"
-			(at 48.26 106.68 0)
+			(at 45.72 106.68 0)
 			(hide yes)
 			(show_name no)
@@
 		)
 		(property "Datasheet" ""
-			(at 48.26 106.68 0)
+			(at 45.72 106.68 0)
 			(hide yes)
 			(show_name no)
@@
 		)
 		(property "Description" "Resistor, small symbol"
-			(at 48.26 106.68 0)
+			(at 45.72 106.68 0)
 			(hide yes)
 			(show_name no)
@@
 					(unit 1)
 				)
+			)
+		)
+	)
+	(symbol
+		(lib_id "HansPinhead:PINHD-1X2")
+		(at 121.92 134.62 90)
+		(unit 1)
+		(body_style 1)
+		(exclude_from_sim no)
+		(in_bom yes)
+		(on_board yes)
+		(in_pos_files yes)
+		(dnp no)
+		(fields_autoplaced yes)
+		(property "Reference" "JP21"
+			(at 121.92 134.62 90)
+			(show_name no)
+			(do_not_autoplace no)
+			(effects
+				(font
+					(size 1.778 1.5113)
+				)
+			)
+		)
+		(property "Value" ""
+			(at 127 140.97 0)
+			(show_name no)
+			(do_not_autoplace no)
+			(effects
+				(font
+					(size 1.778 1.5113)
+				)
+				(justify left bottom)
+			)
+		)
+		(property "Footprint" "HansPinhead:1X02"
+			(at 121.92 134.62 0)
+			(hide yes)
+			(show_name no)
+			(do_not_autoplace no)
+			(effects
+				(font
+					(size 1.27 1.27)
+				)
+			)
+		)
+		(property "Datasheet" ""
+			(at 121.92 134.62 0)
+			(hide yes)
+			(show_name no)
+			(do_not_autoplace no)
+			(effects
+				(font
+					(size 1.27 1.27)
+				)
+			)
+		)
+		(property "Description" "PIN HEADER"
+			(at 121.92 134.62 0)
+			(hide yes)
+			(show_name no)
+			(do_not_autoplace no)
+			(effects
+				(font
+					(size 1.27 1.27)
+				)
+			)
+		)
+		(pin "2"
+		)
+		(pin "1"
+		)
+		(instances
+			(project "v1sch"
+				(path "/cb43fcea-ef29-416a-91e4-99943f7eb9f2/2d477eab-e9a7-46fd-afba-90ac8d8360ce"
+					(reference "JP21")
+					(unit 1)
+				)
