File: v1sch.kicad_pcb (KiCad board)
At the start: 6 copper layers, 100 x 175 mm, 437 parts, among them Q1 APM4953_C5185739, Q10 BSS123, Q11 BSS123, Q12 BC817, Q13 BSS123, Q14 BSS123, Q15 BSS84, Q16 APM4953_C5185739, Q17 BSS123, Q18 BC817, Q19 BC817, Q2 APM4953_C5185739, Q21 BC857, Q22 BC857, Q23 BC817, Q24 BC857, Q25 BC817, Q26 BC857, Q28 BSS123, Q29 BSS123, Q30 BSS123, Q31 BSS123, Q32 BSS123, Q33 BSS123, Q7 BSS123, Q8 BSS123, Q9 BSS123, SW10 TS1701-CZ55HBS, SW11 TS1701-CZ55HBS, SW12 TS1701-CZ55HBS, SW13 TS1701-CZ55HBS, SW6 TS1701-CZ55HBS, SW7 TS1701-CZ55HBS, SW8 TS1701-CZ55HBS, SW9 TS1701-CZ55HBS, U1 STM32G474VETx, U10 SN74CBT3253, U11 SN74CBT3253, U12 TLV9062xD, U13 PCM1821QRTERQ1, U14 NE5532, U15 UAD8C05L01_C3001951, U16 UAD8C05L01_C3001951, U17 161N-4BVS11, U18 161N-4BVS11, U19 LM1084IT-5.0G, U2 DSC1003DL2-008.0000T, U20 UAD8C05L01_C3001951, U21 UAD8C05L01_C3001951, U22 UAD8C05L01_C3001951, U23 UAD8C05L01_C3001951, U24 UAD8C05L01_C3001951, U3 UAD8C05L01_C3001951, U4 UZ1085L-33-TN3-R, U5 UCC27524D, U6 UCC27524D, U7 MC74ACT541DTR2G, U8 MC74ACT541DTR2G, U9 TLV9062xD

Commit message: Update rev1 PCB and schematics with existing project libraries
Parts:
- added JP21: ~, HansPinhead:1X02, F.Cu at (67.6, 22.2)
- moved R107 0.52 mm to (70.5, 18.5)
- moved R1 0.22 mm to (61.4, 144.5)
- moved C64 0.08 mm to (72.4, 65.9)
Connections:
- Q2 pad 5: VIN -> Net-(JP21-Pad1)
- Q2 pad 6: VIN -> Net-(JP21-Pad1)
Routing:
- net Net-(JP21-Pad1): track 0.00 -> 30.9 mm, vias 0 -> 3
- net GND: track 228.4 -> 249.3 mm, vias 664 -> 676
- net VIN: track 491.5 -> 478.6 mm, vias 14 -> 11
- net TX_BIAS: track 81.0 -> 83.9 mm
- net Net-(Q16-G1): track 36.5 -> 34.4 mm
- net Net-(U18-CC1): track 138.1 -> 140.1 mm
- net 3.3V: track 668.4 -> 666.8 mm
- net ADC_VIN: track 81.1 -> 79.7 mm
- net Net-(C34-Pad1): track 42.5 -> 43.5 mm
- net Net-(U11-1B1): track 56.8 -> 55.9 mm
- net Net-(Q31-G): track 263.0 -> 262.1 mm
- net Net-(U5-OUTB): track 89.7 -> 89.0 mm
- net Net-(Q33-G): track 265.2 -> 265.8 mm
Other:
- board text added: "S-HF SPARTACUS REV2"
- board text removed: "SDHFX"
- board text removed: "SPARTACUS REV1"
